File: wifi-geiger-counter.kicad_sch (KiCad schematic)
At the start: 15 parts, among them J1 TYPE-C-31-M-12, J2 S2B-PH-K-S-GW, U1 TP4056, U3 AP2112K-3.3TRG1

Commit message: MCU
Parts:
- added C5: 10u, lcsc:WIFIM-SMD_ESP32-C3-MINI-1, symbol Device:C
- added C6: 100n, lcsc:WIFIM-SMD_ESP32-C3-MINI-1, symbol Device:C
- added C7: 1u, lcsc:WIFIM-SMD_ESP32-C3-MINI-1, symbol Device:C
- added R6, R7, R8, R9: 10k, lcsc:SOT-25-5_L2.9-W1.6-P0.95-LS2.8-BL, symbol Device:R
- added SW1: RESET, Button_Switch_SMD:SW_SPST_CK_KMS2xxGP, symbol Switch:SW_Push
- added SW2: BOOT, Button_Switch_SMD:SW_SPST_CK_KMS2xxGP, symbol Switch:SW_Push
- added U2: ESP32-C3-MINI-1-N4, lcsc:WIFIM-SMD_ESP32-C3-MINI-1, symbol lcsc:ESP32-C3-MINI-1-N4
Connections:
- net +3V3: now also C5.1, C6.1, R6.1, R7.1, R8.1, R9.1, U2.3 (3V3)
- net GND: now also C5.2, C6.2, C7.1, SW1.2, SW2.2, U2.1 (GND), U2.11 (GND), U2.14 (GND), U2.2 (GND), U2.36 (GND), U2.37 (GND), U2.38 (GND), U2.39 (GND), U2.40 (GND), U2.41 (GND), U2.42 (GND), U2.43 (GND), U2.44 (GND), U2.45 (GND), U2.46 (GND), U2.47 (GND), U2.48 (GND), U2.49 (GND), U2.50 (GND), U2.51 (GND), U2.52 (GND), U2.53 (GND)
- net USB_DN: now also U2.26 (IO18)
- net USB_DP: now also U2.27 (IO19)
- new net: R9.2, U2.22 (IO8)
- new net BOOT: R7.2, SW2.1, U2.23 (IO9)
- new net BUZZER: U2.19 (IO5)
- new net EN: C7.2, R6.2, SW1.1, U2.8 (EN)
- new net HV_FB: U2.12 (IO0)
- new net HV_PWM: U2.18 (IO4)
- new net IO2: R8.2, U2.5 (IO2)
- new net PULSE: U2.13 (IO1)
- no-connect marks 3 -> 23
Other:
- moved on the sheet: C1, C2, C3, C4, D1, D2, J1, J2, R1, R2, R3, R4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

Commit message: 400V circuit
Parts:
- added C10, C8, C9: CC1206KKX7RCBB103, lcsc:C1206, symbol lcsc:CC1206KKX7RCBB103
- added C11: 100n, lcsc:WIFIM-SMD_ESP32-C3-MINI-1, symbol Device:C
- added D3, D4, D5: US1M_C83962, lcsc:SMA_L4.3-W2.6-LS5.2-RD, symbol lcsc:US1M_C83962
- added L1: FNR6045S103KT, lcsc:IND-SMD_L6.0-W6.0_FNR60XXS, symbol lcsc:FNR6045S103KT
- added Q1: MMBTA42_C8515, lcsc:SOT-23-3_L2.9-W1.3-P1.90-LS2.4-BR, symbol lcsc:MMBTA42_C8515
- added R10: 1k, lcsc:SOT-25-5_L2.9-W1.6-P0.95-LS2.8-BL, symbol Device:R
- added R11: 10k, lcsc:SOT-25-5_L2.9-W1.6-P0.95-LS2.8-BL, symbol Device:R
- added R12: 220k, lcsc:SOT-25-5_L2.9-W1.6-P0.95-LS2.8-BL, symbol Device:R
- added R13, R14, R15, R16, R17, R18, R19, R20, R21, R22: 10M, lcsc:SOT-25-5_L2.9-W1.6-P0.95-LS2.8-BL, symbol Device:R
Connections:
- net GND: now also C10.2, C11.2, C8.2, Q1.2 (E), R11.1, R12.2
- net HV_FB: now also C11.1, R12.1, R22.2
- net HV_PWM: now also R10.1
- net VBAT: now also L1.1
- new net: Q1.1 (B), R10.2, R11.2
- new net: R15.2, R16.1
- new net: R16.2, R17.1
- new net: R20.2, R21.1
- new net: R21.2, R22.1
- new net: R14.2, R15.1
- new net: R17.2, R18.1
- new net: R18.2, R19.1
- new net: R19.2, R20.1
- new net: R13.2, R14.1
- new net HV: C10.1, D5.1 (C), R13.1
- new net HV1: C8.1, D3.1 (C), D4.2 (A)
- new net HV_X: C9.2, D4.1 (C), D5.2 (A)
- new net SW: C9.1, D3.2 (A), L1.2, Q1.3 (C)

Commit message: add protections, schematic clean
Parts:
- added BZ1: MLT-8530, symbol Device:Buzzer
- added D6: 1N4148W, symbol Device:D
- added D7: SMF5.0A, symbol Device:D_TVS
- added D8: 3.3V, symbol Device:D_Zener
- added D9: LED, symbol Device:LED
- added J3: SBM-20, symbol Connector_Generic:Conn_01x02
- added Q2, Q3: MMBT3904, Package_TO_SOT_SMD:SOT-23, symbol Transistor_BJT:MMBT3904
- added R23: 4.7M, symbol Device:R
- added R24: 100k, symbol Device:R
- added R25, R26, R28: 10k, Package_TO_SOT_SMD:SOT-23, symbol Device:R
- added R27, R29, R30: 1k, Package_TO_SOT_SMD:SOT-23, symbol Device:R
- added U4: USBLC6-2SC6, Package_TO_SOT_SMD:SOT-23-6, symbol Power_Protection:USBLC6-2SC6
Connections:
- net +3V3: now also BZ1.1 (+), D6.1 (K), R26.1
- net BUZZER: now also R27.1
- net GND: now also D7.1 (A1), D8.2 (A), D9.2 (A), Q2.2 (E), Q3.2 (E), R24.1, R28.1, U4.2 (GND)
- net HV: now also R23.1
- net IO2: now also R30.1
- net PULSE: now also Q2.3 (C), R26.2, R29.1; no longer U2.13 (IO1)
- net USB_DN: now also U4.3 (I/O2), U4.4 (I/O2)
- net USB_DP: now also U4.1 (I/O1), U4.6 (I/O1)
- net VBUS: now also D7.2 (A2), U4.5 (VBUS)
- new net: D9.1 (K), R30.2
- new net: J3.1 (Pin_1), R23.2
- new net: Q3.1 (B), R27.2, R28.2
- new net: Q2.1 (B), R25.2
- new net BZ_DRV: BZ1.2 (-), D6.2 (A), Q3.3 (C)
- new net PULSE_SAFE: D8.1 (K), R29.2, U2.13 (IO1)
- new net TUBE_K: J3.2 (Pin_2), R24.2, R25.1
