File: wifi-geiger-counter.kicad_sch (KiCad schematic)
At the start: 64 parts, among them J1 TYPE-C-31-M-12, J2 S2B-PH-K-S-GW, J3 SBM-20, Q1 MMBTA42_C8515, Q2 MMBT3904, Q3 MMBT3904, SW1 RESET, SW2 BOOT, U1 TP4056, U2 ESP32-C3-MINI-1-N4, U3 AP2112K-3.3TRG1, U4 USBLC6-2SC6

Commit message: assign footprints, import into pcb editor
Parts:
- BZ1: footprint (none) -> Buzzer_Beeper:Buzzer_Murata_PKMCS0909E
- C1, C2, C3, C4: footprint (none) -> Capacitor_SMD:C_0805_2012Metric
- C11, C5, C6, C7: footprint lcsc:WIFIM-SMD_ESP32-C3-MINI-1 -> Capacitor_SMD:C_0805_2012Metric
- D1, D2, D9: footprint (none) -> LED_SMD:LED_0805_2012Metric
- D6: footprint (none) -> Diode_SMD:D_SOD-123
- D7: footprint (none) -> Diode_SMD:D_SOD-123F
- D8: footprint (none) -> Diode_SMD:D_SOD-323
- J3: footprint (none) -> Connector_PinHeader_2.54mm:PinHeader_1x02_P2.54mm_Vertical
- R1, R10, R11, R12, R2, R3, R4, R5, R6, R7, R8, R9: footprint lcsc:SOT-25-5_L2.9-W1.6-P0.95-LS2.8-BL -> Resistor_SMD:R_0805_2012Metric
- R13, R14, R15, R16, R17, R18, R19, R20, R21, R22: footprint lcsc:SOT-25-5_L2.9-W1.6-P0.95-LS2.8-BL -> Resistor_SMD:R_1206_3216Metric
- R23: footprint (none) -> Resistor_SMD:R_1206_3216Metric
- R24: footprint (none) -> Resistor_SMD:R_0805_2012Metric
- R25, R26, R27, R28, R29, R30: footprint Package_TO_SOT_SMD:SOT-23 -> Resistor_SMD:R_0805_2012Metric
Changed lines of the file:
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@@
 			)
 		)
-		(property "Footprint" "lcsc:SOT-25-5_L2.9-W1.6-P0.95-LS2.8-BL"
+		(property "Footprint" "Resistor_SMD:R_0805_2012Metric"
 			(at 44.958 251.46 90)
 			(hide yes)
@@
 			)
 		)
-		(property "Footprint" ""
+		(property "Footprint" "Capacitor_SMD:C_0805_2012Metric"
 			(at 235.9152 45.72 0)
 			(hide yes)
@@
 			)
 		)
-		(property "Footprint" "lcsc:SOT-25-5_L2.9-W1.6-P0.95-LS2.8-BL"
+		(property "Footprint" "Resistor_SMD:R_1206_3216Metric"
 			(at 49.53 274.828 90)
 			(hide yes)
@@
 			)
 		)
-		(property "Footprint" ""
+		(property "Footprint" "LED_SMD:LED_0805_2012Metric"
 			(at 261.62 106.68 0)
 			(hide yes)
@@
 			)
 		)
-		(property "Footprint" ""
+		(property "Footprint" "Resistor_SMD:R_0805_2012Metric"
 			(at 184.15 133.858 90)
 			(hide yes)
@@
 			)
 		)
-		(property "Footprint" ""
+		(property "Footprint" "Diode_SMD:D_SOD-123"
 			(at 149.86 123.19 0)
 			(hide yes)
@@
 			)
 		)
-		(property "Footprint" "Package_TO_SOT_SMD:SOT-23"
+		(property "Footprint" "Resistor_SMD:R_0805_2012Metric"
 			(at 252.73 104.648 90)
 			(hide yes)
@@
 			)
 		)
-		(property "Footprint" "lcsc:SOT-25-5_L2.9-W1.6-P0.95-LS2.8-BL"
+		(property "Footprint" "Resistor_SMD:R_0805_2012Metric"
 			(at 34.798 251.46 90)
 			(hide yes)
@@
 			)
 		)
-		(property "Footprint" "lcsc:SOT-25-5_L2.9-W1.6-P0.95-LS2.8-BL"
+		(property "Footprint" "Resistor_SMD:R_1206_3216Metric"
 			(at 87.63 274.828 90)
 			(hide yes)
@@
 			)
 		)
-		(property "Footprint" "lcsc:WIFIM-SMD_ESP32-C3-MINI-1"
+		(property "Footprint" "Capacitor_SMD:C_0805_2012Metric"
 			(at 386.08 87.3252 0)
 			(hide yes)
@@
 			)
 		)
-		(property "Footprint" "lcsc:SOT-25-5_L2.9-W1.6-P0.95-LS2.8-BL"
+		(property "Footprint" "Resistor_SMD:R_0805_2012Metric"
 			(at 313.69 136.398 90)
 			(hide yes)
@@
 			)
 		)
-		(property "Footprint" ""
+		(property "Footprint" "Connector_PinHeader_2.54mm:PinHeader_1x02_P2.54mm_Vertical"
 			(at 173.99 167.64 0)
 			(hide yes)
@@
 			)
 		)
-		(property "Footprint" "lcsc:SOT-25-5_L2.9-W1.6-P0.95-LS2.8-BL"
+		(property "Footprint" "Resistor_SMD:R_1206_3216Metric"
 			(at 41.91 274.828 90)
 			(hide yes)
@@
 			)
 		)
-		(property "Footprint" ""
+		(property "Footprint" "Capacitor_SMD:C_0805_2012Metric"
 			(at 114.6048 38.1 0)
 			(hide yes)
@@
 			)
 		)
-		(property "Footprint" "lcsc:WIFIM-SMD_ESP32-C3-MINI-1"
+		(property "Footprint" "Capacitor_SMD:C_0805_2012Metric"
 			(at 380.6952 69.85 0)
 			(hide yes)
@@
 			)
 		)
-		(property "Footprint" "lcsc:SOT-25-5_L2.9-W1.6-P0.95-LS2.8-BL"
+		(property "Footprint" "Resistor_SMD:R_0805_2012Metric"
 			(at 373.38 113.538 90)
 			(hide yes)
@@
 			)
 		)
-		(property "Footprint" "lcsc:SOT-25-5_L2.9-W1.6-P0.95-LS2.8-BL"
+		(property "Footprint" "Resistor_SMD:R_1206_3216Metric"
 			(at 57.15 274.828 90)
 			(hide yes)
@@
 			)
 		)
-		(property "Footprint" "lcsc:SOT-25-5_L2.9-W1.6-P0.95-LS2.8-BL"
+		(property "Footprint" "Resistor_SMD:R_1206_3216Metric"
 			(at 64.77 274.828 90)
 			(hide yes)
@@
 			)
 		)
-		(property "Footprint" ""
+		(property "Footprint" "LED_SMD:LED_0805_2012Metric"
 			(at 160.02 43.18 0)
 			(hide yes)
@@
 			)
 		)
-		(property "Footprint" "Package_TO_SOT_SMD:SOT-23"
+		(property "Footprint" "Resistor_SMD:R_0805_2012Metric"
 			(at 144.018 148.59 90)
 			(hide yes)
@@
 			)
 		)
-		(property "Footprint" "lcsc:SOT-25-5_L2.9-W1.6-P0.95-LS2.8-BL"
+		(property "Footprint" "Resistor_SMD:R_0805_2012Metric"
 			(at 107.95 281.178 90)
 			(hide yes)
@@
 			)
 		)
-		(property "Footprint" "lcsc:SOT-25-5_L2.9-W1.6-P0.95-LS2.8-BL"
+		(property "Footprint" "Resistor_SMD:R_1206_3216Metric"
 			(at 72.39 274.828 90)
 			(hide yes)
@@
 			)
 		)
-		(property "Footprint" ""
+		(property "Footprint" "Capacitor_SMD:C_0805_2012Metric"
 			(at 248.6152 45.72 0)
 			(hide yes)
@@
 			)
 		)
-		(property "Footprint" "Package_TO_SOT_SMD:SOT-23"
+		(property "Footprint" "Resistor_SMD:R_0805_2012Metric"
 			(at 204.47 156.718 90)
 			(hide yes)
@@
 			)
 		)
-		(property "Footprint" "lcsc:SOT-25-5_L2.9-W1.6-P0.95-LS2.8-BL"
+		(property "Footprint" "Resistor_SMD:R_1206_3216Metric"
 			(at 95.25 274.828 90)
 			(hide yes)
@@
 			)
 		)
-		(property "Footprint" ""
+		(property "Footprint" "Resistor_SMD:R_1206_3216Metric"
 			(at 172.212 158.75 90)
 			(hide yes)
@@
 			)
 		)
-		(property "Footprint" "lcsc:SOT-25-5_L2.9-W1.6-P0.95-LS2.8-BL"
+		(property "Footprint" "Resistor_SMD:R_0805_2012Metric"
 			(at 62.23 43.688 90)
 			(hide yes)
@@
 			)
 		)
-		(property "Footprint" "lcsc:SOT-25-5_L2.9-W1.6-P0.95-LS2.8-BL"
+		(property "Footprint" "Resistor_SMD:R_0805_2012Metric"
 			(at 210.82 60.198 90)
 			(hide yes)
@@
 			)
 		)
-		(property "Footprint" ""
+		(property "Footprint" "Capacitor_SMD:C_0805_2012Metric"
 			(at 133.0452 45.72 0)
 			(hide yes)
@@
 			)
 		)
-		(property "Footprint" "lcsc:SOT-25-5_L2.9-W1.6-P0.95-LS2.8-BL"
+		(property "Footprint" "Resistor_SMD:R_1206_3216Metric"
 			(at 34.29 274.828 90)
 			(hide yes)
@@
 			)
 		)
-		(property "Footprint" "Package_TO_SOT_SMD:SOT-23"
+		(property "Footprint" "Resistor_SMD:R_0805_2012Metric"
 			(at 323.85 58.928 90)
 			(hide yes)
@@
 			)
 		)
-		(property "Footprint" "lcsc:SOT-25-5_L2.9-W1.6-P0.95-LS2.8-BL"
+		(property "Footprint" "Resistor_SMD:R_1206_3216Metric"
 			(at 80.01 274.828 90)
 			(hide yes)
@@
 			)
 		)
-		(property "Footprint" "lcsc:SOT-25-5_L2.9-W1.6-P0.95-LS2.8-BL"
+		(property "Footprint" "Resistor_SMD:R_0805_2012Metric"
 			(at 167.64 37.338 90)
 			(hide yes)
@@
 			)
 		)
-		(property "Footprint" ""
+		(property "Footprint" "Diode_SMD:D_SOD-323"
 			(at 332.74 60.96 0)
 			(hide yes)
@@
 			)
 		)
-		(property "Footprint" "Package_TO_SOT_SMD:SOT-23"
+		(property "Footprint" "Resistor_SMD:R_0805_2012Metric"
 			(at 214.122 138.43 90)
 			(hide yes)
@@
 			)
 		)
-		(property "Footprint" "lcsc:SOT-25-5_L2.9-W1.6-P0.95-LS2.8-BL"
+		(property "Footprint" "Resistor_SMD:R_0805_2012Metric"
 			(at 62.23 58.928 90)
 			(hide yes)
@@
 			)
 		)
-		(property "Footprint" "lcsc:SOT-25-5_L2.9-W1.6-P0.95-LS2.8-BL"
+		(property "Footprint" "Resistor_SMD:R_0805_2012Metric"
 			(at 303.53 93.218 90)
 			(hide yes)
@@
 			)
 		)
-		(property "Footprint" "lcsc:SOT-25-5_L2.9-W1.6-P0.95-LS2.8-BL"
+		(property "Footprint" "Resistor_SMD:R_0805_2012Metric"
 			(at 373.38 88.138 90)
 			(hide yes)
@@
 			)
 		)
-		(property "Footprint" ""
+		(property "Footprint" "Diode_SMD:D_SOD-123F"
 			(at 274.32 72.39 0)
 			(hide yes)
@@
 			)
 		)
-		(property "Footprint" "lcsc:SOT-25-5_L2.9-W1.6-P0.95-LS2.8-BL"
+		(property "Footprint" "Resistor_SMD:R_0805_2012Metric"
 			(at 167.64 44.958 90)
 			(hide yes)
@@
 			)
 		)
-		(property "Footprint" ""
+		(property "Footprint" "Buzzer_Beeper:Buzzer_Murata_PKMCS0909E"
 			(at 151.765 104.14 90)
 			(hide yes)
@@
 			)
 		)
-		(property "Footprint" "lcsc:WIFIM-SMD_ESP32-C3-MINI-1"
+		(property "Footprint" "Capacitor_SMD:C_0805_2012Metric"
 			(at 137.16 279.7048 0)
 			(hide yes)
@@
 			)
 		)
-		(property "Footprint" "lcsc:SOT-25-5_L2.9-W1.6-P0.95-LS2.8-BL"
+		(property "Footprint" "Resistor_SMD:R_1206_3216Metric"
 			(at 26.67 274.828 90)
 			(hide yes)
@@
 			)
 		)
-		(property "Footprint" "lcsc:WIFIM-SMD_ESP32-C3-MINI-1"
+		(property "Footprint" "Capacitor_SMD:C_0805_2012Metric"
 			(at 365.4552 69.85 0)
 			(hide yes)
@@
 			)
 		)
-		(property "Footprint" ""
+		(property "Footprint" "LED_SMD:LED_0805_2012Metric"
 			(at 160.02 35.56 0)
 			(hide yes)
@@
 			)
 		)
-		(property "Footprint" "Package_TO_SOT_SMD:SOT-23"
+		(property "Footprint" "Resistor_SMD:R_0805_2012Metric"
 			(at 138.43 137.668 90)
 			(hide yes)
