File: pcb/wifi-geiger-counter.kicad_pcb (KiCad board)
At the start: 2 copper layers, 95 x 55 mm, 64 parts, among them J1 TYPE-C-31-M-12, J2 S2B-PH-K-S-GW, J3 SBM-20, Q1 MMBTA42_C8515, Q2 MMBT3904, Q3 MMBT3904, SW1 RESET, SW2 BOOT, U1 TP4056, U2 ESP32-C3-MINI-1-N4, U3 AP2112K-3.3TRG1, U4 USBLC6-2SC6

Commit message: Fix PCB issues, address design feedback
Fixing the BOM.csv, README, folder structuring and design flaws

- Moved KiCad things, libraries, gerbers, etc. into pcb/
- Added BOM.csv and improved README
- Fixed TVS polarity, status LED, buzzer footprint
- Fixed USB-C connector orientation
- Fixed net class patterns and clearance
- ADC/PWM/conversion factor firmware fixes
Parts:
- BZ1: footprint Buzzer_Beeper:Buzzer_Murata_PKMCS0909E -> lcsc:BUZ-SMD_4P-L8.5-W8.5-P8.50-BR
- D2: value GREEN -> YELLOW
- D7: value SMF5.0A -> SMF5.0CA
- J3: value SBM-20 -> M4011
- R3: value 2k -> 2.2k
- moved BZ1 3.77 mm to (54.7, 166.8), turned to 90 degrees
- moved J1 1.96 mm to (52.1, 125.1), turned to -90 degrees
Connections:
- net Net-(J3-Pin_1) renamed /TUBE_A
- D9 pad 2: GND -> +3V3
Routing:
- net GND: track 16.7 -> 66.8 mm, vias 8 -> 10
- net /USB_DP: track 84.5 -> 76.6 mm, vias 7 -> 6
- net +3V3: track 151.3 -> 159.2 mm, vias 6 -> 7
- net /BZ_DRV: track 11.8 -> 18.7 mm
- net Net-(J1-CC2): track 15.9 -> 22.3 mm, vias 0 -> 2
- net /USB_DN: track 85.0 -> 78.8 mm
- net Net-(J1-CC1): track 15.7 -> 10.2 mm
- net Net-(Q1-B): track 9.67 -> 13.5 mm
- net /VBUS: track 65.8 -> 64.6 mm
