File: pcb/wifi-geiger-counter.kicad_sch (KiCad schematic)
At the start: 64 parts, among them J1 TYPE-C-31-M-12, J2 S2B-PH-K-S-GW, J3 SBM-20, Q1 MMBTA42_C8515, Q2 MMBT3904, Q3 MMBT3904, SW1 RESET, SW2 BOOT, U1 TP4056, U2 ESP32-C3-MINI-1-N4, U3 AP2112K-3.3TRG1, U4 USBLC6-2SC6

Commit message: Fix PCB issues, address design feedback
Fixing the BOM.csv, README, folder structuring and design flaws

- Moved KiCad things, libraries, gerbers, etc. into pcb/
- Added BOM.csv and improved README
- Fixed TVS polarity, status LED, buzzer footprint
- Fixed USB-C connector orientation
- Fixed net class patterns and clearance
- ADC/PWM/conversion factor firmware fixes
Parts:
- BZ1: footprint Buzzer_Beeper:Buzzer_Murata_PKMCS0909E -> lcsc:BUZ-SMD_4P-L8.5-W8.5-P8.50-BR
- D2: value GREEN -> YELLOW
- D7: value SMF5.0A -> SMF5.0CA
- J3: value SBM-20 -> M4011
- R3: value 2k -> 2.2k
- SW1, SW2: now not fitted
Connections:
- net +3V3: now also D9.2 (A)
- net GND: no longer D9.2 (A)
- net TUBE_A: now reaches J3.1 (Pin_1), R23.2
Other:
- moved on the sheet: R23
Changed lines of the file:
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@@
 	(wire
 		(pts
+			(xy 173.99 160.02) (xy 173.99 162.56)
+		)
+		(stroke
+			(width 0)
+			(type default)
+		)
+	)
+	(wire
+		(pts
 			(xy 340.36 106.68) (xy 340.36 104.14)
 		)
@@
 	)
 	(label "HV"
-		(at 173.99 154.94 0)
+		(at 173.99 152.4 0)
 		(effects
 			(font
@@
 		)
 	)
+	(label "TUBE_A"
+		(at 173.99 161.29 0)
+		(effects
+			(font
+				(size 1.27 1.27)
+			)
+			(justify left bottom)
+		)
+	)
 	(label "EN"
 		(at 308.61 99.06 180)
@@
 		(on_board yes)
 		(in_pos_files yes)
-		(dnp no)
+		(dnp yes)
 		(fields_autoplaced yes)
 		(property "Reference" "SW2"
@@
 			)
 		)
-		(property "Value" "SBM-20"
+		(property "Value" "M4011"
 			(at 176.53 168.9099 90)
 			(show_name no)
@@
 			)
 		)
-		(property "Value" "GREEN"
+		(property "Value" "YELLOW"
 			(at 158.242 40.894 0)
 			(show_name no)
@@
 	(symbol
 		(lib_id "power:GND")
-		(at 261.62 110.49 0)
-		(unit 1)
-		(body_style 1)
-		(exclude_from_sim no)
-		(in_bom yes)
-		(on_board yes)
-		(in_pos_files yes)
-		(dnp no)
-		(fields_autoplaced yes)
-		(property "Reference" "#PWR056"
-			(at 261.62 116.84 0)
-			(hide yes)
-			(show_name no)
-			(do_not_autoplace no)
-			(effects
-				(font
-					(size 1.27 1.27)
-				)
-			)
-		)
-		(property "Value" "GND"
-			(at 261.62 115.57 0)
-			(show_name no)
-			(do_not_autoplace no)
-			(effects
-				(font
-					(size 1.27 1.27)
-				)
-			)
-		)
-		(property "Footprint" ""
-			(at 261.62 110.49 0)
-			(hide yes)
-			(show_name no)
-			(do_not_autoplace no)
-			(effects
-				(font
-					(size 1.27 1.27)
-				)
-			)
-		)
-		(property "Datasheet" ""
-			(at 261.62 110.49 0)
-			(hide yes)
-			(show_name no)
-			(do_not_autoplace no)
-			(effects
-				(font
-					(size 1.27 1.27)
-				)
-			)
-		)
-		(property "Description" "Power symbol creates a global label with name \"GND\" , ground"
-			(at 261.62 110.49 0)
-			(hide yes)
-			(show_name no)
-			(do_not_autoplace no)
-			(effects
-				(font
-					(size 1.27 1.27)
-				)
-			)
-		)
-		(pin "1"
-		)
-		(instances
-			(project "wifi-geiger-counter"
-				(path "/ea347852-16b2-4adf-b0d8-c3ef89e2ab6b"
-					(reference "#PWR056")
-					(unit 1)
-				)
-			)
-		)
-	)
-	(symbol
-		(lib_id "power:GND")
 		(at 38.1 240.03 90)
 		(unit 1)
@@
 	(symbol
 		(lib_id "Device:R")
-		(at 173.99 158.75 0)
+		(at 173.99 156.21 0)
 		(unit 1)
 		(body_style 1)
@@
 		(fields_autoplaced yes)
 		(property "Reference" "R23"
-			(at 176.53 157.4799 0)
+			(at 176.53 154.9399 0)
 			(show_name no)
 			(do_not_autoplace no)
@@
 		)
 		(property "Value" "4.7M"
-			(at 176.53 160.0199 0)
+			(at 176.53 157.4799 0)
 			(show_name no)
 			(do_not_autoplace no)
@@
 		)
 		(property "Footprint" "Resistor_SMD:R_1206_3216Metric"
-			(at 172.212 158.75 90)
+			(at 172.212 156.21 90)
 			(hide yes)
 			(show_name no)
@@
 		)
 		(property "Datasheet" ""
-			(at 173.99 158.75 0)
+			(at 173.99 156.21 0)
 			(hide yes)
 			(show_name no)
@@
 		)
 		(property "Description" "Resistor"
-			(at 173.99 158.75 0)
+			(at 173.99 156.21 0)
 			(hide yes)
 			(show_name no)
@@
 			)
 		)
-		(property "Value" "2k"
+		(property "Value" "2.2k"
 			(at 210.82 56.134 90)
 			(show_name no)
@@
 		(on_board yes)
 		(in_pos_files yes)
-		(dnp no)
+		(dnp yes)
 		(fields_autoplaced yes)
 		(property "Reference" "SW1"
@@
 	)
 	(symbol
+		(lib_id "power:+3V3")
+		(at 261.62 110.49 180)
+		(unit 1)
+		(body_style 1)
+		(exclude_from_sim no)
+		(in_bom yes)
+		(on_board yes)
+		(in_pos_files yes)
+		(dnp no)
+		(fields_autoplaced yes)
+		(property "Reference" "#PWR056"
+			(at 261.62 106.68 0)
+			(hide yes)
+			(show_name no)
+			(do_not_autoplace no)
+			(effects
+				(font
+					(size 1.27 1.27)
+				)
+			)
+		)
+		(property "Value" "+3V3"
+			(at 261.62 115.57 0)
+			(show_name no)
+			(do_not_autoplace no)
+			(effects
+				(font
+					(size 1.27 1.27)
+				)
+			)
+		)
+		(property "Footprint" ""
+			(at 261.62 110.49 0)
+			(hide yes)
+			(show_name no)
+			(do_not_autoplace no)
+			(effects
+				(font
+					(size 1.27 1.27)
+				)
+			)
+		)
+		(property "Datasheet" ""
+			(at 261.62 110.49 0)
+			(hide yes)
+			(show_name no)
+			(do_not_autoplace no)
+			(effects
+				(font
+					(size 1.27 1.27)
+				)
+			)
+		)
+		(property "Description" "Power symbol creates a global label with name \"+3V3\""
+			(at 261.62 110.49 0)
+			(hide yes)
+			(show_name no)
+			(do_not_autoplace no)
+			(effects
+				(font
+					(size 1.27 1.27)
+				)
+			)
+		)
+		(pin "1"
+		)
+		(instances
+			(project "wifi-geiger-counter"
+				(path "/ea347852-16b2-4adf-b0d8-c3ef89e2ab6b"
+					(reference "#PWR056")
+					(unit 1)
+				)
+			)
+		)
+	)
+	(symbol
 		(lib_id "Device:R")
 		(at 167.64 35.56 90)
@@
 			)
 		)
-		(property "Value" "SMF5.0A"
+		(property "Value" "SMF5.0CA"
 			(at 276.86 73.6599 90)
 			(show_name no)
@@
 			)
 		)
-		(property "Footprint" "Buzzer_Beeper:Buzzer_Murata_PKMCS0909E"
+		(property "Footprint" "lcsc:BUZ-SMD_4P-L8.5-W8.5-P8.50-BR"
 			(at 151.765 104.14 90)
 			(hide yes)
